File: backplane/backplane.sch (KiCad schematic (older format))
At the start: 59 parts

Commit message: Iter 2019-10-07
Parts:
- U?: symbol WAVGAT_CAN:WAVGAT_CAN -> backplane-rescue:WAVGAT_CAN-WAVGAT_CAN
Changed lines of the file:
@@
 	8950 4850 8950 4950
 $Comp
-L WAVGAT_CAN:WAVGAT_CAN U?
+L backplane-rescue:WAVGAT_CAN-WAVGAT_CAN U?
 U 1 1 5E9A99C5
 P 11400 3600
