File: hardware/backplane/backplane.kicad_pcb (KiCad board)
At the start: 2 copper layers, 100 x 49 mm, 59 parts, among them J1 Conn_01x02_Male, J10 DB9_Male, J11 Conn_01x02_Male, J12 Conn_01x02_Male, J2 RJ45_LED, J3 Conn_01x02_Male, J4 Conn_01x02_Male, J5 RJ45_LED, J6 Raspberry_Pi_2_3, J7 RJ45_LED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

Commit message: Finish backplane release candidate.
Parts:
- removed J11, J12, J3, J4: Conn_01x02_Male, Connector_PinHeader_2.54mm:PinHeader_1x02_P2.54mm_Vertical
- removed J7, J8: RJ45_LED, Connector_RJ:RJ45_BEL_SS74301-00x_Vertical
- removed R21, R22, R25, R26: 10K, Resistor_SMD:R_0603_1608Metric_Pad1.05x0.95mm_HandSolder
- added J13: Conn_01x08_Male, Connector_PinHeader_2.54mm:PinHeader_1x08_P2.54mm_Vertical, F.Cu at (169.3, 117.5)
- C1, C2, C9, J2, J5, R2, R31, R5: moved to F.Cu
- J1: value Conn_01x02_Male -> Conn_01x04_Male; footprint Connector_PinHeader_2.54mm:PinHeader_1x02_P2.54mm_Vertical -> Connector_PinHeader_2.54mm:PinHeader_1x04_P2.54mm_Vertical
- J10: value DB9_Male -> Conn_02x10_Odd_Even; footprint Connector_Dsub:DSUB-9_Male_Horizontal_P2.77x2.54mm_EdgePinOffset9.40mm -> Connector_PinHeader_2.54mm:PinHeader_2x10_P2.54mm_Vertical
- J6: footprint Connector_PinSocket_2.54mm:PinSocket_2x20_P2.54mm_Vertical -> Connector_PinHeader_2.54mm:PinHeader_2x20_P2.54mm_Vertical
- J9: value DB9_Female -> Conn_02x10_Odd_Even; footprint Connector_Dsub:DSUB-9_Female_Horizontal_P2.77x2.54mm_EdgePinOffset9.40mm -> Connector_PinHeader_2.54mm:PinHeader_2x10_P2.54mm_Vertical
- R1, R29, R3, R30, R6, R8, R9, U5: moved to B.Cu
- R13, R14: value 560R -> 0R; moved to B.Cu
- R23, R24: value 560R -> 0R
- moved R3 135.3 mm to (160.2, 71.1)
- moved C6 129.0 mm to (137.1, 79.4)
- moved C8 112.6 mm to (131.6, 82.6)
- moved C7 111.4 mm to (123.7, 82.5)
- moved R1 108.1 mm to (156.9, 76.8), turned to 90 degrees
- moved R16 101.6 mm to (155.9, 108.3)
- moved C5 99.0 mm to (132.6, 77.5)
- moved R23 91.7 mm to (125.2, 90.2), turned to 270 degrees
- moved D1 90.0 mm to (88.3, 76.5), turned to 90 degrees
- moved J6 84.7 mm to (91.2, 74.7), turned to 90 degrees
- moved R5 79.4 mm to (83.8, 79.9)
- moved C1 78.3 mm to (84.6, 76.5)
- moved U1 77.2 mm to (94.6, 80.7), turned to 180 degrees
- moved R4 74.8 mm to (88.3, 73.0), turned to 90 degrees
- moved J1 74.5 mm to (146.9, 72.2), turned to 0 degrees
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Connections:
- J1 pad 1: /CANBUS_HIGH -> Net-(J1-Pad1)
- J10 pad 1: Net-(J10-Pad1) -> GND
- J10 pad 2: /CANBUS_LOW -> /CANBUS_HIGH
- J10 pad 3: VCC -> /CANBUS_LOW
- J10 pad 4: /SCL -> GND
- J10 pad 5: +12V -> GND
- J10 pad 6: GND -> /SDA
- J10 pad 7: /CANBUS_HIGH -> /SCL
- J10 pad 8: /SDA -> GND
- J10 pad 9: VCC -> +12V
- J6 pad 10: Net-(J6-Pad10) -> (no net)
- J6 pad 11: Net-(J6-Pad11) -> (no net)
- J6 pad 12: Net-(J6-Pad12) -> Net-(J1-Pad1)
- J6 pad 13: Net-(J6-Pad13) -> (no net)
- J6 pad 18: Net-(J6-Pad18) -> (no net)
- J6 pad 22: Net-(J6-Pad22) -> (no net)
- J6 pad 24: Net-(J6-Pad24) -> (no net)
- J6 pad 26: Net-(J6-Pad26) -> (no net)
- J6 pad 27: Net-(J6-Pad27) -> (no net)
- J6 pad 28: Net-(J6-Pad28) -> (no net)
- J6 pad 29: Net-(J6-Pad29) -> (no net)
- J6 pad 31: Net-(J6-Pad31) -> (no net)
- J6 pad 32: Net-(J6-Pad32) -> Net-(J1-Pad2)
- J6 pad 33: Net-(J6-Pad33) -> Net-(J1-Pad3)
- J6 pad 35: Net-(J6-Pad35) -> (no net)
- J6 pad 36: Net-(J6-Pad36) -> (no net)
- J6 pad 37: Net-(J6-Pad37) -> (no net)
- J6 pad 38: Net-(J6-Pad38) -> (no net)
- J6 pad 40: Net-(J6-Pad40) -> (no net)
- J6 pad 7: Net-(J6-Pad7) -> (no net)
- J6 pad 8: Net-(J6-Pad8) -> (no net)
- J9 pad 1: Net-(J9-Pad1) -> GND
- J9 pad 2: /CANBUS_LOW -> /CANBUS_HIGH
- J9 pad 3: VCC -> /CANBUS_LOW
- J9 pad 4: /SCL -> GND
- J9 pad 5: +12V -> GND
- J9 pad 6: GND -> /SDA
- J9 pad 7: /CANBUS_HIGH -> /SCL
- J9 pad 8: /SDA -> GND
- J9 pad 9: VCC -> +12V
- R13 pad 1: VCC -> /SCL
- R13 pad 2: Net-(J7-Pad10) -> Net-(R13-Pad2)
- R14 pad 1: VCC -> Net-(R14-Pad1)
- R14 pad 2: Net-(J7-Pad12) -> /SDA
- R2 pad 1: Net-(J1-Pad2) -> /CANBUS_HIGH
- R23 pad 1: VCC -> /CANBUS_LOW
- R23 pad 2: Net-(J8-Pad10) -> Net-(R23-Pad2)
- R24 pad 1: VCC -> Net-(R24-Pad1)
- R24 pad 2: Net-(J8-Pad12) -> /CANBUS_HIGH
- R31 pad 1: Net-(J11-Pad2) -> /CANBUS_HIGH
- R32 pad 1: Net-(J12-Pad2) -> /CANBUS_LOW
- R5 pad 1: Net-(J3-Pad2) -> /CANBUS_LOW
- U1 pad 1: /SCL -> Net-(R13-Pad2)
- U1 pad 8: /SDA -> Net-(R14-Pad1)
- U3 pad 1: Net-(U3-Pad1) -> (no net)
- U3 pad 4: Net-(U3-Pad4) -> (no net)
- U4 pad 11: Net-(U4-Pad11) -> (no net)
- U4 pad 14: Net-(U4-Pad14) -> (no net)
- U4 pad 19: Net-(U4-Pad19) -> (no net)
- U4 pad 20: Net-(U4-Pad20) -> (no net)
- U4 pad 23: WIRE_GOOD_2 -> (no net)
- U4 pad 24: WIRE_GOOD_3 -> (no net)
- U4 pad 27: MODULE_GOOD_2 -> (no net)
- U4 pad 28: MODULE_GOOD_3 -> (no net)
- U5 pad J1_1: Net-(U5-PadJ1_1) -> (no net)
- U5 pad J1_2: Net-(U5-PadJ1_2) -> (no net)
- U5 pad J3_1: /CANBUS_HIGH -> Net-(R24-Pad1)
- U5 pad J3_2: /CANBUS_LOW -> Net-(R23-Pad2)
- U5 pad J4_1: Net-(U5-PadJ4_1) -> (no net)
Routing:
- net VCC: track 25.8 -> 306.0 mm, vias 1 -> 11
- net +3V3: track 0.00 -> 175.5 mm, vias 0 -> 7
- net /CANBUS_LOW: track 0.00 -> 135.7 mm, vias 0 -> 2
- net /SCL: track 0.00 -> 135.2 mm, vias 0 -> 2
- net /SDA: track 0.00 -> 131.8 mm, vias 0 -> 4
- net /CANBUS_HIGH: track 0.00 -> 128.2 mm, vias 0 -> 2
- net GND: track 12.7 -> 137.1 mm, vias 3 -> 22
- net +12V: track 0.00 -> 117.0 mm, vias 0 -> 1
- net WIRE_GOOD_1: track 0.00 -> 87.6 mm, vias 0 -> 1
- net MODULE_GOOD_1: track 0.00 -> 78.0 mm, vias 0 -> 4
- net WIRE_GOOD_0: track 0.00 -> 50.2 mm, vias 0 -> 3
- net Net-(J1-Pad1): track 0.00 -> 44.5 mm
- net Net-(J6-Pad16): track 0.00 -> 30.6 mm
- net MODULE_GOOD_0: track 0.00 -> 29.1 mm, vias 0 -> 5
- net Net-(R24-Pad1): track 0.00 -> 23.5 mm
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- added copper zone on B.Cu, net GND
Other:
- board size 100 x 49 mm -> 100 x 50 mm
