File: hardware/backplane/backplane.sch (KiCad schematic (older format))
At the start: 59 parts

Commit message: Refactor PCB files from root folder -> hardware/
Parts:
- removed J?: Barrel_Jack, symbol Connector:Barrel_Jack
- added J4: Conn_01x02_Male, Connector_PinHeader_2.54mm:PinHeader_1x02_P2.54mm_Vertical, symbol Connector:Conn_01x02_Male
- C1, C2, C3, C4, C5, C6, C7, C8, C9: renamed from C?; footprint (none) -> Capacitor_SMD:C_0603_1608Metric_Pad1.05x0.95mm_HandSolder
- D1: renamed from D?; footprint (none) -> LED_SMD:LED_0603_1608Metric_Pad1.05x0.95mm_HandSolder
- J1, J11, J12, J3: renamed from J?; footprint (none) -> Connector_PinHeader_2.54mm:PinHeader_1x02_P2.54mm_Vertical
- J10: renamed from J?; footprint (none) -> Connector_Dsub:DSUB-9_Male_Horizontal_P2.77x2.54mm_EdgePinOffset9.40mm
- J2, J5, J7, J8: renamed from J?; footprint (none) -> Connector_RJ:RJ45_BEL_SS74301-00x_Vertical
- J6: renamed from J?; footprint (none) -> Connector_PinHeader_2.54mm:PinHeader_2x20_P2.54mm_Vertical
- J9: renamed from J?; footprint (none) -> Connector_Dsub:DSUB-9_Female_Horizontal_P2.77x2.54mm_EdgePinOffset9.40mm
- R1, R10, R11, R12, R13, R14, R15, R16, R17, R18, R19, R2, R20, R21, R22, R23, R24, R25, R26, R27, R28, R29, R3, R30, R31, R32, R4, R5, R6, R7, R8, R9: renamed from R?; footprint (none) -> Resistor_SMD:R_0603_1608Metric_Pad1.05x0.95mm_HandSolder
- U5: renamed from U?; footprint (none) -> WAVGAT_CAN:WAVGAT_CAN
- gave numbers to parts that had none: 4
Connections:
- wire segments 394 -> 416

Commit message: Finish backplane release candidate.
Parts:
- removed J1, J11, J12, J3, J4: Conn_01x02_Male, Connector_PinHeader_2.54mm:PinHeader_1x02_P2.54mm_Vertical, symbol Connector:Conn_01x02_Male
- removed J10: DB9_Male, Connector_Dsub:DSUB-9_Male_Horizontal_P2.77x2.54mm_EdgePinOffset9.40mm, symbol Connector:DB9_Male
- removed J7, J8: RJ45_LED, Connector_RJ:RJ45_BEL_SS74301-00x_Vertical, symbol Connector:RJ45_LED
- removed J9: DB9_Female, Connector_Dsub:DSUB-9_Female_Horizontal_P2.77x2.54mm_EdgePinOffset9.40mm, symbol Connector:DB9_Female
- removed R21, R22, R25, R26: 10K, Resistor_SMD:R_0603_1608Metric_Pad1.05x0.95mm_HandSolder, symbol Device:R
- added J1: Conn_01x04_Male, Connector_PinHeader_2.54mm:PinHeader_1x04_P2.54mm_Vertical, symbol Connector:Conn_01x04_Male
- added J10, J9: Conn_02x10_Odd_Even, Connector_PinHeader_2.54mm:PinHeader_2x10_P2.54mm_Vertical, symbol backplane-rescue:Conn_02x10_Odd_Even-Connector_Generic
- added J13: Conn_01x08_Male, Connector_PinHeader_2.54mm:PinHeader_1x08_P2.54mm_Vertical, symbol Connector:Conn_01x08_Male
- C1, C2, C3, C4, C5, C6, C7, C8, C9: symbol Device:C -> backplane-rescue:C-Device
- D1: symbol Device:LED -> backplane-rescue:LED-Device
- J2, J5: symbol Connector:RJ45_LED -> backplane-rescue:RJ45_LED-Connector
- J6: symbol Connector:Raspberry_Pi_2_3 -> backplane-rescue:Raspberry_Pi_2_3-Connector
- R1, R10, R11, R12, R15, R16, R17, R18, R19, R2, R20, R27, R28, R29, R3, R30, R31, R32, R4, R5, R6, R7, R8, R9: symbol Device:R -> backplane-rescue:R-Device
- R13, R14, R23, R24: value 560R -> 0R
- U1, U2, U3: symbol Logic_LevelTranslator:TXB0102DCU -> backplane-rescue:TXB0102DCU-Logic_LevelTranslator
- U4: symbol Interface_Expansion:MCP23017_SO -> backplane-rescue:MCP23017_SO-Interface_Expansion
Connections:
- net labels removed: MODULE_GOOD_2, MODULE_GOOD_3, WIRE_GOOD_2, WIRE_GOOD_3
- wire segments 416 -> 365

Commit message: Reorient RJ45 connectors in backplane, make interrupt pins accessible in IO Expanders
Parts:
- added J3: Conn_01x02_Male-Connector, Connector_PinHeader_2.54mm:PinHeader_1x02_P2.54mm_Vertical, symbol backplane-rescue:Conn_01x02_Male-Connector
Connections:
- wire segments 365 -> 371
Changed lines of the file:
@@
 Wire Wire Line
 	2850 4500 2600 4500
+$Comp
+L backplane-rescue:Conn_01x02_Male-Connector J3
+U 1 1 5DC6B261
+P 7100 13900
+F 0 "J3" H 7208 14081 50  0000 C CNN
+F 1 "Conn_01x02_Male-Connector" H 7208 13990 50  0000 C CNN
+F 2 "Connector_PinHeader_2.54mm:PinHeader_1x02_P2.54mm_Vertical" H 7100 13900 50  0001 C CNN
+F 3 "" H 7100 13900 50  0001 C CNN
+	1    7100 13900
+	1    0    0    -1
+$EndComp
+Wire Wire Line
+	7300 13900 7650 13900
+Wire Wire Line
+	7650 13900 7650 14100
+Wire Wire Line
+	7650 14100 7700 14100
+Wire Wire Line
+	7300 14000 7600 14000
+Wire Wire Line
+	7600 14000 7600 14200
+Wire Wire Line
+	7600 14200 7700 14200
 $EndSCHEMATC

Commit message: New backplane schematic
Parts:
- removed C3, C4, C5, C6, C7, C8: 0.1uF, Capacitor_SMD:C_0603_1608Metric_Pad1.05x0.95mm_HandSolder, symbol backplane-rescue:C-Device
- removed C9: 4n7, Capacitor_SMD:C_0603_1608Metric_Pad1.05x0.95mm_HandSolder, symbol backplane-rescue:C-Device
- removed J1: Conn_01x04_Male, Connector_PinHeader_2.54mm:PinHeader_1x04_P2.54mm_Vertical, symbol Connector:Conn_01x04_Male
- removed J10, J9: Conn_02x10_Odd_Even, Connector_PinHeader_2.54mm:PinHeader_2x10_P2.54mm_Vertical, symbol backplane-rescue:Conn_02x10_Odd_Even-Connector_Generic
- removed J3: Conn_01x02_Male-Connector, Connector_PinHeader_2.54mm:PinHeader_1x02_P2.54mm_Vertical, symbol backplane-rescue:Conn_01x02_Male-Connector
- removed J5: RJ45_LED, Connector_RJ:RJ45_BEL_SS74301-00x_Vertical, symbol backplane-rescue:RJ45_LED-Connector
- removed R19, R20, R27, R28: 10K, Resistor_SMD:R_0603_1608Metric_Pad1.05x0.95mm_HandSolder, symbol backplane-rescue:R-Device
- removed R24: 0R, Resistor_SMD:R_0603_1608Metric_Pad1.05x0.95mm_HandSolder, symbol Device:R
- removed R29, R30, R6, R7: 4K7, Resistor_SMD:R_0603_1608Metric_Pad1.05x0.95mm_HandSolder, symbol backplane-rescue:R-Device
- removed R31, R32: 60R, Resistor_SMD:R_0603_1608Metric_Pad1.05x0.95mm_HandSolder, symbol backplane-rescue:R-Device
- removed R8, R9: 560R, Resistor_SMD:R_0603_1608Metric_Pad1.05x0.95mm_HandSolder, symbol backplane-rescue:R-Device
- removed U1, U2, U3: TXB0102DCU, Package_SO:VSSOP-8_2.4x2.1mm_P0.5mm, symbol backplane-rescue:TXB0102DCU-Logic_LevelTranslator
- removed U5: WAVGAT_CAN, WAVGAT_CAN:WAVGAT_CAN, symbol backplane-rescue:WAVGAT_CAN-WAVGAT_CAN
- added C1: 10u, Capacitor_SMD:C_0805_2012Metric_Pad1.15x1.40mm_HandSolder, symbol Device:C
- added C10, C2, C3: 100n, Capacitor_SMD:C_0603_1608Metric_Pad1.05x0.95mm_HandSolder, symbol Device:C
- added C11, C9: 22p, Capacitor_SMD:C_0603_1608Metric_Pad1.05x0.95mm_HandSolder, symbol Device:C
- added C12, C8: 470n, Capacitor_SMD:C_0805_2012Metric_Pad1.15x1.40mm_HandSolder, symbol Device:C
- added C14: 4n7, Capacitor_SMD:C_0603_1608Metric_Pad1.05x0.95mm_HandSolder, symbol Device:C
- added C4, C5, C6: 1u, Capacitor_SMD:C_0805_2012Metric_Pad1.15x1.40mm_HandSolder, symbol Device:C
- added C7: 47u, Capacitor_THT:CP_Radial_D5.0mm_P2.00mm, symbol Device:CP
- added D2: LED, LED_SMD:LED_0603_1608Metric_Pad1.05x0.95mm_HandSolder, symbol Device:LED
- added J1, J3: Screw_Terminal_01x02, TerminalBlock_Phoenix:TerminalBlock_Phoenix_PT-1,5-2-5.0-H_1x02_P5.00mm_Horizontal, symbol Connector:Screw_Terminal_01x02
- added J10, J11, J6: RJ45_LED, Connector_RJ:RJ45_BEL_SS74301-00x_Vertical, symbol Connector:RJ45_LED_Shielded
- added J4: Screw_Terminal_01x03, TerminalBlock_Phoenix:TerminalBlock_Phoenix_PT-1,5-3-5.0-H_1x03_P5.00mm_Horizontal, symbol Connector:Screw_Terminal_01x03
- added J8, J9: Conn_02x08_Odd_Even, Connector_PinHeader_2.54mm:PinHeader_2x08_P2.54mm_Vertical, symbol Connector_Generic:Conn_02x08_Odd_Even
- added Q1, Q2, Q3, Q4: Q_NMOS_GSD, Package_TO_SOT_SMD:SOT-23_Handsoldering, symbol Device:Q_NMOS_GSD
- added R1, R12, R15, R2, R5, R6, R7, R8, R9: 10k, Resistor_SMD:R_0603_1608Metric_Pad1.05x0.95mm_HandSolder, symbol Device:R
- added R11: 2k, Resistor_SMD:R_0603_1608Metric_Pad1.05x0.95mm_HandSolder, symbol Device:R
- added R16, R17, R3, R4: 0R, Resistor_SMD:R_0603_1608Metric_Pad1.05x0.95mm_HandSolder, symbol Device:R
- added R19: 60R, Resistor_SMD:R_0603_1608Metric_Pad1.05x0.95mm_HandSolder, symbol Device:R
- added R21, R25, R27, R28, R29, R30: 560R, Resistor_SMD:R_0603_1608Metric_Pad1.05x0.95mm_HandSolder, symbol Device:R
- added U1: TJA1051T, Package_SO:SOIC-8_3.9x4.9mm_P1.27mm, symbol Interface_CAN_LIN:TJA1051T
- added U2: MCP2515-xSO, Package_SO:SOIC-18W_7.5x11.6mm_P1.27mm, symbol Interface_CAN_LIN:MCP2515-xSO
- added U3: PAM8403, Package_SO:SOIC-16_3.9x9.9mm_P1.27mm, symbol ProjectChips:PAM8403
- added Y1: 8MHz, Crystal:Crystal_HC49-U_Vertical, symbol Device:Crystal
- C13: renamed from C1; symbol backplane-rescue:C-Device -> Device:C
- C15: renamed from C2; value 0.1uF -> 100n; symbol backplane-rescue:C-Device -> Device:C
- D1: symbol backplane-rescue:LED-Device -> Device:LED
- J2: renamed from J6; footprint Connector_PinHeader_2.54mm:PinHeader_2x20_P2.54mm_Vertical -> Connector_PinSocket_2.54mm:PinSocket_2x20_P2.54mm_Vertical; symbol backplane-rescue:Raspberry_Pi_2_3-Connector -> Connector:Raspberry_Pi_2_3
- J5: renamed from J2; symbol backplane-rescue:RJ45_LED-Connector -> Connector:RJ45_LED_Shielded
- J7: renamed from J13; value Conn_01x08_Male -> Conn_01x08_Female; footprint Connector_PinHeader_2.54mm:PinHeader_1x08_P2.54mm_Vertical -> Connector_PinSocket_2.54mm:PinSocket_1x08_P2.54mm_Vertical; symbol Connector:Conn_01x08_Male -> Connector:Conn_01x08_Female
- R10: renamed from R4; symbol backplane-rescue:R-Device -> Device:R
- R13, R14: value 0R -> 10k
- R18: renamed from R5; symbol backplane-rescue:R-Device -> Device:R
- R20: renamed from R1; symbol backplane-rescue:R-Device -> Device:R
- R22: renamed from R2; symbol backplane-rescue:R-Device -> Device:R
- R23: value 0R -> 60R
- R24: renamed from R3; symbol backplane-rescue:R-Device -> Device:R
- R26: renamed from R16; symbol backplane-rescue:R-Device -> Device:R
- R31: renamed from R10; symbol backplane-rescue:R-Device -> Device:R
- R32: renamed from R11; symbol backplane-rescue:R-Device -> Device:R
- R33: renamed from R12; symbol backplane-rescue:R-Device -> Device:R
- R34: renamed from R15; symbol backplane-rescue:R-Device -> Device:R
- R35: renamed from R17; symbol backplane-rescue:R-Device -> Device:R
- R36: renamed from R18; symbol backplane-rescue:R-Device -> Device:R
- U4: symbol backplane-rescue:MCP23017_SO-Interface_Expansion -> Interface_Expansion:MCP23017_SO
Connections:
- net labels added: AUDIO_L, AUDIO_R, CAN_CS, CAN_H, CAN_INT, CAN_L, CAN_MISO, CAN_MOSI, CAN_SCLK, MCP23017_INT, MODULE_ENABLE_0, MODULE_ENABLE_1, MODULE_ENABLE_2, MODULE_ENABLE_3, MODULE_READY_0, MODULE_READY_1, MODULE_READY_2, MODULE_READY_3, SCL_3V3, SDA_3V3, SPKR_L+, SPKR_L-, SPKR_R+, SPKR_R-
- net labels removed: CANBUS_HIGH, CANBUS_LOW, MODULE_GOOD_0, MODULE_GOOD_1, WIRE_GOOD_0, WIRE_GOOD_1
- wire segments 371 -> 349
- no-connect marks 0 -> 10
Other:
- note added: "Audio amplifier (optional, only with RasPi)"
- note added: "CAN module (only with RasPi)"
- note added: "CAN termination (only in ends of chain)"
- note added: "Chaining connectors"
- note added: "GPIO expander"
- note added: "I2C level shifter + pullup (only with RasPi)"
- note added: "Module connectors"
- note added: "Power LEDs"
- note added: "Power input\n(only one in chain)"
- note added: "Raspberry Pi (only one in chain)"
- note added: "TODO:\novervoltage protection?\ninput caps?"

Commit message: First revision of PCB layout for backplane v2
Parts:
- removed C1: 10u, Capacitor_SMD:C_0805_2012Metric_Pad1.15x1.40mm_HandSolder, symbol Device:C
- removed J7: Conn_01x08_Female, Connector_PinSocket_2.54mm:PinSocket_1x08_P2.54mm_Vertical, symbol Connector:Conn_01x08_Female
- removed R20, R21, R24, R25, R27, R28, R29, R30: 560R, Resistor_SMD:R_0603_1608Metric_Pad1.05x0.95mm_HandSolder, symbol Device:R
- added C12: 100u, Capacitor_THT:CP_Radial_D7.5mm_P2.50mm, symbol Device:CP
- added D1: LED, LED_THT:LED_D3.0mm, symbol Device:LED
- added J7: Conn_02x08_Top_Bottom, Connector_PinSocket_2.54mm:PinSocket_2x08_P2.54mm_Vertical, symbol Connector_Generic:Conn_02x08_Odd_Even
- added R10: 270R, Resistor_SMD:R_0603_1608Metric_Pad1.05x0.95mm_HandSolder, symbol Device:R
- D2: renamed from D1; footprint LED_SMD:LED_0603_1608Metric_Pad1.05x0.95mm_HandSolder -> LED_THT:LED_D3.0mm
- D3: renamed from D2; footprint LED_SMD:LED_0603_1608Metric_Pad1.05x0.95mm_HandSolder -> LED_THT:LED_D3.0mm
- J10, J11, J5, J6: footprint Connector_RJ:RJ45_BEL_SS74301-00x_Vertical -> RJ45_5224:RJ45_5224; symbol Connector:RJ45_LED_Shielded -> Connector:RJ45_Shielded
- renumbered C2 to C1, C11 to C10, C12 to C11, C3 to C2, C4 to C3, C5 to C4, C6 to C5, C7 to C6, C8 to C7, C9 to C8, C10 to C9, R10 to R11, R11 to R12, R12 to R13, R13 to R14, R14 to R15, R15 to R16, R16 to R17, R17 to R18, R18 to R19, R19 to R20, R22 to R23, R23 to R24, R26 to R27, R31 to R32, R32 to R33, R33 to R34, R34 to R35, R35 to R36, R36 to R37
Connections:
- net +3V3: now also R10.1
- net GND: now also J8.15 (Pin_15), J8.16 (Pin_16), J9.15 (Pin_15), J9.16 (Pin_16), U1.8 (S), C12.2, D1.1 (K), J7.10 (Pin_10), J7.12 (Pin_12), J7.14 (Pin_14), J7.16 (Pin_16), J7.2 (Pin_2), J7.4 (Pin_4), J7.6 (Pin_6), J7.8 (Pin_8)
- net MODULE_ENABLE_0: now also U4.22 (GPA1); no longer J5.9, U4.21 (GPA0)
- net MODULE_ENABLE_1: now also U4.24 (GPA3); no longer J6.9, U4.22 (GPA1)
- net MODULE_ENABLE_2: now also U4.26 (GPA5); no longer J10.9, U4.23 (GPA2)
- net MODULE_ENABLE_3: now also U4.28 (GPA7); no longer J11.9, U4.24 (GPA3)
- net MODULE_READY_0: now also U4.21 (GPA0); no longer J5.11, U4.25 (GPA4)
- net MODULE_READY_1: now also U4.23 (GPA2); no longer J6.11, U4.26 (GPA5)
- net MODULE_READY_2: now also U4.25 (GPA4); no longer J10.11, U4.27 (GPA6)
- net MODULE_READY_3: now also U4.27 (GPA6); no longer J11.11, U4.28 (GPA7)
- net VCC: now also C12.1
- net at U4.1 (GPB0): now also J7.1 (Pin_1)
- net GPIO_A0: now reaches R36.1, R37.1, U4.15 (A0)
- net GPIO_A1: now reaches R34.1, R35.1, U4.16 (A1)
- net GPIO_A2: now reaches R32.1, R33.1, U4.17 (A2)
- net at U4.2 (GPB1): now also J7.3 (Pin_3)
- net at U4.3 (GPB2): now also J7.5 (Pin_5)
- net at U4.4 (GPB3): now also J7.7 (Pin_7)
- net at U4.5 (GPB4): now also J7.9 (Pin_9)
- net at U4.6 (GPB5): now also J7.11 (Pin_11)
- net at U4.7 (GPB6): now also J7.13 (Pin_13)
- net at U4.8 (GPB7): now also J7.15 (Pin_15)
- new net: D1.2 (A), R10.2
- no-connect marks 10 -> 9
Other:
- note added: "TODO:\novervoltage protection?"
- note removed: "TODO:\novervoltage protection?\ninput caps?"
- moved on the sheet: D2, D3, J4, R11, R12

Commit message: Backplane PCB: add audio filter circuit
Parts:
- added C14, C15: 100n, Capacitor_SMD:C_0603_1608Metric_Pad1.05x0.95mm_HandSolder, symbol Device:C
- added C17, C18: 47u, Capacitor_THT:CP_Radial_D5.0mm_P2.00mm, symbol Device:C
- added J8: Conn_01x03, Connector_PinHeader_2.54mm:PinHeader_1x03_P2.54mm_Vertical, symbol Connector_Generic:Conn_01x03
- added R28, R29, R30, R31: 100R, Resistor_SMD:R_0603_1608Metric_Pad1.05x0.95mm_HandSolder, symbol Device:R
- J3: renamed from J5; value RJ45_LED -> RJ45
- J4: renamed from J10; value RJ45_LED -> RJ45
- J5: renamed from J6; value RJ45_LED -> RJ45
- J6: renamed from J11; value RJ45_LED -> RJ45
- renumbered C15 to C1, C3 to C10, C13 to C11, C4 to C12, C5 to C13, C6 to C16, C14 to C19, C8 to C2, C10 to C3, C2 to C4, C1 to C5, C12 to C6, C9 to C8, C11 to C9, J2 to J1, J1 to J10, J3 to J11, J9 to J12, J7 to J2, J4 to J7, J8 to J9, Q3 to Q1, Q4 to Q2, Q1 to Q3, Q2 to Q4, R13 to R1, R37 to R10, R15 to R11, R16 to R12, R18 to R13, R9 to R14, R1 to R15, R6 to R16, R2 to R17, R7 to R18, R10 to R19, R32 to R2, R11 to R20, R3 to R21, R4 to R22, R12 to R23, R5 to R24, R8 to R25, R19 to R26, R23 to R27, R33 to R3, R20 to R32, R24 to R33, R14 to R4, R34 to R5, R17 to R6, R35 to R7, R27 to R8, R36 to R9, U4 to U1, U1 to U3, U3 to U4
Connections:
- net AUDIO_L: now also C17.1, J8.1 (Pin_1); no longer J1.32 (PWM0/GPIO12)
- net AUDIO_R: now also C18.1, J8.3 (Pin_3); no longer J1.33 (PWM1/GPIO13)
- net GND: now also C14.2, C15.2, J8.2 (Pin_2), R30.2, R31.2
- new net: C14.1, C17.2, R28.1, R30.1
- new net: C15.1, C18.2, R29.1, R31.1
- new net PWM0: J1.32 (PWM0/GPIO12), R28.2
- new net PWM1: J1.33 (PWM1/GPIO13), R29.2
Other:
- note added: "Audio filtering (only with RasPi Zero)"

Commit message: Backplane PCB: add overvoltage protection, remove some 0Rs, some reorganization
Parts:
- removed Q3, Q4: Q_NMOS_GSD, Package_TO_SOT_SMD:SOT-23_Handsoldering, symbol Device:Q_NMOS_GSD
- removed R15, R16, R17, R18: 10k, Resistor_SMD:R_0603_1608Metric_Pad1.05x0.95mm_HandSolder, symbol Device:R
- removed R21, R22: 0R, Resistor_SMD:R_0603_1608Metric_Pad1.05x0.95mm_HandSolder, symbol Device:R
- added C20: 100n, Capacitor_SMD:C_0603_1608Metric_Pad1.05x0.95mm_HandSolder, symbol Device:C
- added D4: BZX384-4V3, symbol Diode:BZX384-xxx
- added Q3, Q4, Q5: ZXMP4A16G, Package_TO_SOT_SMD:SOT-223-3_TabPin2, symbol Transistor_FET:ZXMP4A16G
- R13, R6: value 0R -> 10k; footprint Resistor_SMD:R_0603_1608Metric_Pad1.05x0.95mm_HandSolder -> (none)
- U3: value TJA1051T -> TJA1051T/3; symbol Interface_CAN_LIN:TJA1051T -> Interface_CAN_LIN:TJA1051T-3
Connections:
- net +3V3: now also U3.5 (VIO), C20.1
- net CAN_H: now also U3.7 (CANH)
- net CAN_L: now also U3.6 (CANL)
- net GND: now also R13.2, C20.2, D4.2 (A), Q3.1 (G)
- net SCL: now also Q1.3 (D), R4.2; no longer R6.1
- net SDA: now also Q2.3 (D), R12.2; no longer R13.1
- net VCC: now also Q5.2 (D); no longer J7.1 (Pin_1)
- net at U2.1 (TXCAN): now also U3.1 (TXD)
- net at U2.2 (RXCAN): now also U3.4 (RXD)
- new net: Q4.2 (D), Q5.1 (G), R13.1
- new net: Q3.3 (S), Q4.3 (S), Q5.3 (S), R6.1
- new net: D4.1 (K), Q4.1 (G), R6.2
- new net +5V: J7.1 (Pin_1), Q3.2 (D)
Other:
- note added: "Power input w/ overvoltage protection\n(only one in chain)"
- note removed: "Power input\n(only one in chain)"
- note removed: "TODO:\novervoltage protection?"
- moved on the sheet: C6

Commit message: Backplane PCB: remove 3.3V from backplane connector
Parts:
- D4: footprint (none) -> Diode_SMD:D_SOD-323_HandSoldering
- R13, R6: footprint (none) -> Resistor_SMD:R_0603_1608Metric_Pad1.05x0.95mm_HandSolder
Connections:
- net +3V3: no longer J12.13 (Pin_13), J12.14 (Pin_14), J9.13 (Pin_13), J9.14 (Pin_14)
- no-connect marks 9 -> 13
Changed lines of the file:
@@
 Wire Wire Line
 	14800 8950 14650 8950
-$Comp
-L power:+3.3V #PWR092
-U 1 1 60811883
-P 15450 9550
-F 0 "#PWR092" H 15450 9400 50  0001 C CNN
-F 1 "+3.3V" V 15465 9678 50  0000 L CNN
-F 2 "" H 15450 9550 50  0001 C CNN
-F 3 "" H 15450 9550 50  0001 C CNN
-	1    15450 9550
-	0    1    1    0
-$EndComp
 Wire Wire Line
 	15300 9250 15450 9250
@@
 	1    15000 9250
 	1    0    0    -1
-$EndComp
-$Comp
-L power:+3.3V #PWR086
-U 1 1 6081186E
-P 14650 9550
-F 0 "#PWR086" H 14650 9400 50  0001 C CNN
-F 1 "+3.3V" V 14665 9678 50  0000 L CNN
-F 2 "" H 14650 9550 50  0001 C CNN
-F 3 "" H 14650 9550 50  0001 C CNN
-	1    14650 9550
-	0    -1   -1   0
 $EndComp
 $Comp
@@
 Wire Wire Line
 	13050 8950 12900 8950
-$Comp
-L power:+3.3V #PWR074
-U 1 1 606EE94C
-P 13700 9550
-F 0 "#PWR074" H 13700 9400 50  0001 C CNN
-F 1 "+3.3V" V 13715 9678 50  0000 L CNN
-F 2 "" H 13700 9550 50  0001 C CNN
-F 3 "" H 13700 9550 50  0001 C CNN
-	1    13700 9550
-	0    1    1    0
-$EndComp
 Wire Wire Line
 	13550 9250 13700 9250
@@
 	1    13250 9250
 	1    0    0    -1
-$EndComp
-$Comp
-L power:+3.3V #PWR065
-U 1 1 5DD05E97
-P 12900 9550
-F 0 "#PWR065" H 12900 9400 50  0001 C CNN
-F 1 "+3.3V" V 12915 9678 50  0000 L CNN
-F 2 "" H 12900 9550 50  0001 C CNN
-F 3 "" H 12900 9550 50  0001 C CNN
-	1    12900 9550
-	0    -1   -1   0
 $EndComp
 $Comp
@@
 F 0 "R6" H 10570 6346 50  0000 L CNN
 F 1 "10k" H 10570 6255 50  0000 L CNN
-F 2 "" V 10430 6300 50  0001 C CNN
+F 2 "Resistor_SMD:R_0603_1608Metric_Pad1.05x0.95mm_HandSolder" V 10430 6300 50  0001 C CNN
 F 3 "~" H 10500 6300 50  0001 C CNN
 	1    10500 6300
@@
 F 0 "D4" V 10454 6880 50  0000 L CNN
 F 1 "BZX384-4V3" V 10545 6880 50  0000 L CNN
-F 2 "" H 10500 6800 50  0001 C CNN
+F 2 "Diode_SMD:D_SOD-323_HandSoldering" H 10500 6800 50  0001 C CNN
 F 3 "~" H 10500 6800 50  0001 C CNN
 	1    10500 6800
@@
 F 0 "R13" H 11620 6996 50  0000 L CNN
 F 1 "10k" H 11620 6905 50  0000 L CNN
-F 2 "" V 11480 6950 50  0001 C CNN
+F 2 "Resistor_SMD:R_0603_1608Metric_Pad1.05x0.95mm_HandSolder" V 11480 6950 50  0001 C CNN
 F 3 "~" H 11550 6950 50  0001 C CNN
 	1    11550 6950
@@
 Wire Wire Line
 	10250 7700 10250 7950
+NoConn ~ 15450 9550
+NoConn ~ 14650 9550
+NoConn ~ 13700 9550
+NoConn ~ 12900 9550
 $EndSCHEMATC
