File: hardware/backplane/backplane.sch (KiCad schematic (older format))
At the start: 73 parts, among them J1 Raspberry_Pi_2_3, J10 Screw_Terminal_01x02, J11 Screw_Terminal_01x02, J12 Conn_02x08_Odd_Even, J2 Conn_02x08_Top_Bottom, J3 RJ45, J4 RJ45, J5 RJ45, J6 RJ45, J7 Screw_Terminal_01x03, J8 Conn_01x03, J9 Conn_02x08_Odd_Even, Q1 Q_NMOS_GSD, Q2 Q_NMOS_GSD, Q3 ZXMP4A16G, Q4 ZXMP4A16G, Q5 ZXMP4A16G, U1 MCP23017_SO, U2 MCP2515-xSO, U3 TJA1051T/3, U4 PAM8403, Y1 8MHz

Commit message: Backplane PCB: thermal pads for power FETs, lots of finishing touches
Parts:
- C1, C11, C14, C15, C19, C2, C20, C3, C4, C5, C8: footprint Capacitor_SMD:C_0603_1608Metric_Pad1.05x0.95mm_HandSolder -> Capacitor_SMD:C_0805_2012Metric_Pad1.15x1.40mm_HandSolder
Changed lines of the file:
@@
 F 0 "C1" V 2798 8100 50  0000 C CNN
 F 1 "100n" V 2889 8100 50  0000 C CNN
-F 2 "Capacitor_SMD:C_0603_1608Metric_Pad1.05x0.95mm_HandSolder" H 3088 7950 50  0001 C CNN
+F 2 "Capacitor_SMD:C_0805_2012Metric_Pad1.15x1.40mm_HandSolder" H 3088 7950 50  0001 C CNN
 F 3 "~" H 3050 8100 50  0001 C CNN
 	1    3050 8100
@@
 F 0 "C5" V 9198 1600 50  0000 C CNN
 F 1 "100n" V 9289 1600 50  0000 C CNN
-F 2 "Capacitor_SMD:C_0603_1608Metric_Pad1.05x0.95mm_HandSolder" H 9488 1450 50  0001 C CNN
+F 2 "Capacitor_SMD:C_0805_2012Metric_Pad1.15x1.40mm_HandSolder" H 9488 1450 50  0001 C CNN
 F 3 "~" H 9450 1600 50  0001 C CNN
 	1    9450 1600
@@
 F 0 "C2" V 4498 2800 50  0000 C CNN
 F 1 "22p" V 4589 2800 50  0000 C CNN
-F 2 "Capacitor_SMD:C_0603_1608Metric_Pad1.05x0.95mm_HandSolder" H 4788 2650 50  0001 C CNN
+F 2 "Capacitor_SMD:C_0805_2012Metric_Pad1.15x1.40mm_HandSolder" H 4788 2650 50  0001 C CNN
 F 3 "~" H 4750 2800 50  0001 C CNN
 	1    4750 2800
@@
 F 0 "C3" V 4900 3100 50  0000 C CNN
 F 1 "22p" V 5000 3100 50  0000 C CNN
-F 2 "Capacitor_SMD:C_0603_1608Metric_Pad1.05x0.95mm_HandSolder" H 4788 2950 50  0001 C CNN
+F 2 "Capacitor_SMD:C_0805_2012Metric_Pad1.15x1.40mm_HandSolder" H 4788 2950 50  0001 C CNN
 F 3 "~" H 4750 3100 50  0001 C CNN
 	1    4750 3100
@@
 F 0 "C4" V 5598 1700 50  0000 C CNN
 F 1 "100n" V 5689 1700 50  0000 C CNN
-F 2 "Capacitor_SMD:C_0603_1608Metric_Pad1.05x0.95mm_HandSolder" H 5888 1550 50  0001 C CNN
+F 2 "Capacitor_SMD:C_0805_2012Metric_Pad1.15x1.40mm_HandSolder" H 5888 1550 50  0001 C CNN
 F 3 "~" H 5850 1700 50  0001 C CNN
 	1    5850 1700
@@
 F 0 "C8" V 12098 2800 50  0000 C CNN
 F 1 "100n" V 12189 2800 50  0000 C CNN
-F 2 "Capacitor_SMD:C_0603_1608Metric_Pad1.05x0.95mm_HandSolder" H 12388 2650 50  0001 C CNN
+F 2 "Capacitor_SMD:C_0805_2012Metric_Pad1.15x1.40mm_HandSolder" H 12388 2650 50  0001 C CNN
 F 3 "~" H 12350 2800 50  0001 C CNN
 	1    12350 2800
@@
 F 0 "C11" H 13265 7846 50  0000 L CNN
 F 1 "4n7" H 13265 7755 50  0000 L CNN
-F 2 "Capacitor_SMD:C_0603_1608Metric_Pad1.05x0.95mm_HandSolder" H 13188 7650 50  0001 C CNN
+F 2 "Capacitor_SMD:C_0805_2012Metric_Pad1.15x1.40mm_HandSolder" H 13188 7650 50  0001 C CNN
 F 3 "~" H 13150 7800 50  0001 C CNN
 	1    13150 7800
@@
 F 0 "C19" H 15365 7846 50  0000 L CNN
 F 1 "4n7" H 15365 7755 50  0000 L CNN
-F 2 "Capacitor_SMD:C_0603_1608Metric_Pad1.05x0.95mm_HandSolder" H 15288 7650 50  0001 C CNN
+F 2 "Capacitor_SMD:C_0805_2012Metric_Pad1.15x1.40mm_HandSolder" H 15288 7650 50  0001 C CNN
 F 3 "~" H 15250 7800 50  0001 C CNN
 	1    15250 7800
@@
 F 0 "C14" H 14000 5250 50  0000 L CNN
 F 1 "100n" H 13900 5150 50  0000 L CNN
-F 2 "Capacitor_SMD:C_0603_1608Metric_Pad1.05x0.95mm_HandSolder" H 14238 5050 50  0001 C CNN
+F 2 "Capacitor_SMD:C_0805_2012Metric_Pad1.15x1.40mm_HandSolder" H 14238 5050 50  0001 C CNN
 F 3 "~" H 14200 5200 50  0001 C CNN
 	1    14200 5200
@@
 F 0 "C15" H 14000 6400 50  0000 L CNN
 F 1 "100n" H 13900 6300 50  0000 L CNN
-F 2 "Capacitor_SMD:C_0603_1608Metric_Pad1.05x0.95mm_HandSolder" H 14238 6200 50  0001 C CNN
+F 2 "Capacitor_SMD:C_0805_2012Metric_Pad1.15x1.40mm_HandSolder" H 14238 6200 50  0001 C CNN
 F 3 "~" H 14200 6350 50  0001 C CNN
 	1    14200 6350
@@
 F 0 "C20" H 8700 2600 50  0000 L CNN
 F 1 "100n" H 8650 2500 50  0000 L CNN
-F 2 "Capacitor_SMD:C_0603_1608Metric_Pad1.05x0.95mm_HandSolder" H 8988 2400 50  0001 C CNN
+F 2 "Capacitor_SMD:C_0805_2012Metric_Pad1.15x1.40mm_HandSolder" H 8988 2400 50  0001 C CNN
 F 3 "~" H 8950 2550 50  0001 C CNN
 	1    8950 2550

Commit message: Backplane PCB: add section field to components
Parts:
- C1, J12, J2, J3, J4, J5, J6, J9, R10, R2, R3, R5, R7, R8, R9, U1: Section (none) -> IO
- C10, C12, C13, C16, C7, C8, C9, J10, J11, J8, R24, R25, U4: Section (none) -> AudioAmp
- C11, C19, R26, R27, R32, R33: Section (none) -> CanTermination
- C14, C15, C17, C18, R28, R29, R30, R31: Section (none) -> AudioFilter
- C2, C20, C3, C4, C5, R14, U2, U3, Y1: Section (none) -> CanModule
- C6, D4, J7, Q3, Q4, Q5, R13, R6: Section (none) -> PowerInput
- D1, J1, Q1, Q2, R1, R11, R12, R19, R4: Section (none) -> RaspberryPi
- D2, D3, R20, R23: Section (none) -> PowerLed

Commit message: Backplane PCB: I2S audio and complete relayout
Parts:
- removed C10: 1u, Capacitor_SMD:C_0805_2012Metric_Pad1.15x1.40mm_HandSolder, symbol Device:C
- removed C16: 47u, Capacitor_THT:CP_Radial_D5.0mm_P2.00mm, symbol Device:CP
- removed C17, C18: 47u, Capacitor_THT:CP_Radial_D5.0mm_P2.00mm, symbol Device:C
- removed C7, C9: 470n, Capacitor_SMD:C_0805_2012Metric_Pad1.15x1.40mm_HandSolder, symbol Device:C
- removed C8: 100n, Capacitor_SMD:C_0805_2012Metric_Pad1.15x1.40mm_HandSolder, symbol Device:C
- removed J8: Conn_01x03, Connector_PinHeader_2.54mm:PinHeader_1x03_P2.54mm_Vertical, symbol Connector_Generic:Conn_01x03
- removed R24, R25: 10k, Resistor_SMD:R_0603_1608Metric_Pad1.05x0.95mm_HandSolder, symbol Device:R
- removed R28, R29, R30, R31: 100R, Resistor_SMD:R_0603_1608Metric_Pad1.05x0.95mm_HandSolder, symbol Device:R
- removed U4: PAM8403, Package_SO:SOIC-16_3.9x9.9mm_P1.27mm, symbol ProjectChips:PAM8403
- added C2: 10u, Capacitor_SMD:C_0805_2012Metric_Pad1.15x1.40mm_HandSolder, symbol Device:C
- added C3: 1u, Capacitor_SMD:C_0805_2012Metric_Pad1.15x1.40mm_HandSolder, symbol Device:C
- added FB1, FB2, FB3, FB4: Ferrite, Capacitor_SMD:C_0805_2012Metric_Pad1.15x1.40mm_HandSolder, symbol Device:Ferrite_Bead_Small
- added R22: 100k, Resistor_SMD:R_0603_1608Metric_Pad1.05x0.95mm_HandSolder, symbol Device:R
- added R23: 330k, Resistor_SMD:R_0603_1608Metric_Pad1.05x0.95mm_HandSolder, symbol Device:R
- added U4, U5: MAX98357AETE, Package_DFN_QFN:TQFN-16-1EP_3x3mm_P0.5mm_EP1.23x1.23mm_ThermalVias, symbol ProjectChips:MAX98357AETE
- C12: value 1u -> 10u
- C13: value 1u -> 100n
- C14: value 100n -> 10u; Section AudioFilter -> AudioAmp
- C15: Section AudioFilter -> AudioAmp
- D1: renamed from D4; value BZX384-4V3 -> BZX384-5V1
- renumbered C6 to C1, C11 to C10, C19 to C11, C2 to C5, C3 to C6, C5 to C7, C20 to C8, C1 to C9, D1 to D2, D2 to D3, D3 to D4, J11 to J10, J2 to J11, J7 to J2, J5 to J4, J4 to J5, J12 to J7, J9 to J8, J10 to J9, R6 to R1, R5 to R10, R7 to R11, R9 to R12, R10 to R13, R8 to R14, R19 to R15, R20 to R16, R23 to R17, R32 to R18, R33 to R19, R13 to R2, R26 to R20, R27 to R21, R14 to R3, R1 to R4, R4 to R5, R11 to R6, R12 to R7, R2 to R8, R3 to R9, U2 to U1, U3 to U2, U1 to U3
Connections:
- net GND: now also C2.2, C3.2, U4.11 (GND), U4.15 (GND), U4.17 (EP), U4.3 (GND), U5.11 (GND), U5.15 (GND), U5.17 (EP), U5.3 (GND)
- net MODULE_ENABLE_0: now also U3.24 (GPA3); no longer U3.22 (GPA1)
- net MODULE_ENABLE_1: now also U3.22 (GPA1); no longer U3.24 (GPA3)
- net MODULE_ENABLE_2: now also U3.28 (GPA7); no longer U3.26 (GPA5)
- net MODULE_ENABLE_3: now also U3.26 (GPA5); no longer U3.28 (GPA7)
- net MODULE_READY_0: now also U3.23 (GPA2); no longer U3.21 (GPA0)
- net MODULE_READY_1: now also U3.21 (GPA0); no longer U3.23 (GPA2)
- net MODULE_READY_2: now also U3.27 (GPA6); no longer U3.25 (GPA4)
- net MODULE_READY_3: now also U3.25 (GPA4); no longer U3.27 (GPA6)
- net SPKR_L+: now also FB1.1
- net SPKR_L-: now also FB3.2
- net SPKR_R+: now also J10.1 (Pin_1), FB2.1; no longer J10.2 (Pin_2)
- net SPKR_R-: now also J10.2 (Pin_2), FB4.2; no longer J10.1 (Pin_1)
- net VCC: now also C14.1, C15.1, C2.1, C3.1, R22.1, R23.1, U4.4 (~SD_MODE), U4.7 (VDD), U4.8 (VDD), U5.7 (VDD), U5.8 (VDD)
- net PCM_BCLK: now reaches J1.12 (GPIO18/PWM0)
- net PCM_BCLK: now also U4.16 (BCLK), U5.16 (BCLK)
- net PCM_LRCLK: now reaches J1.35 (GPIO19/MISO1)
- net PCM_LRCLK: now also U4.14 (LRCLK), U5.14 (LRCLK)
- net PCM_DOUT: now reaches J1.40 (GPIO21/SCLK1)
- net PCM_DOUT: now also U4.1 (DIN), U5.1 (DIN)
- net PWM0: no longer names the net of J1.32 (PWM0/GPIO12)
- net PWM1: no longer names the net of J1.33 (PWM1/GPIO13)
- new net: FB3.1, U4.10 (OUTN)
- new net: FB1.2, U4.9 (OUTP)
- new net: FB4.1, U5.10 (OUTN)
- new net: R23.2, U5.4 (~SD_MODE)
- new net: FB2.2, U5.9 (OUTP)
- new net AUDIO_GAIN: R22.2, U4.2 (GAIN_SLOT), U5.2 (GAIN_SLOT)
- no-connect marks 13 -> 11
Other:
- note added: "Power LEDs\n3.3V only with RasPi\nRest on all boards"
- note removed: "Audio filtering (only with RasPi Zero)"
- note removed: "Power LEDs"
- moved on the sheet: C1, C4, C5, C6, C7, C8, D1, D2, D3, D4, J10, J2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
