File: hardware/password/module_shared.sch (KiCad schematic (older format))
At the start: 7 parts, among them J1 RJ45_Shielded, U1 WAVGAT_CAN

Commit message: Password PCB: change display polarity
Parts:
- R1, R2: footprint Resistor_SMD:R_0603_1608Metric_Pad1.05x0.95mm_HandSolder -> Resistor_SMD:R_0603_1608Metric_Pad0.98x0.95mm_HandSolder
Changed lines of the file:
@@
 F 0 "R2" H 1770 3746 50  0000 L CNN
 F 1 "560R" H 1770 3655 50  0000 L CNN
-F 2 "Resistor_SMD:R_0603_1608Metric_Pad1.05x0.95mm_HandSolder" V 1630 3700 50  0001 C CNN
+F 2 "Resistor_SMD:R_0603_1608Metric_Pad0.98x0.95mm_HandSolder" V 1630 3700 50  0001 C CNN
 F 3 "~" H 1700 3700 50  0001 C CNN
 	1    1700 3700
@@
 F 0 "R1" H 1770 2546 50  0000 L CNN
 F 1 "560R" H 1770 2455 50  0000 L CNN
-F 2 "Resistor_SMD:R_0603_1608Metric_Pad1.05x0.95mm_HandSolder" V 1630 2500 50  0001 C CNN
+F 2 "Resistor_SMD:R_0603_1608Metric_Pad0.98x0.95mm_HandSolder" V 1630 2500 50  0001 C CNN
 F 3 "~" H 1700 2500 50  0001 C CNN
 	1    1700 2500
